Commit message: minor update: new functions, bugs (#83)
* DefDict Math update *add

* Fixed kinematics bug for scaler legs

* changed to use relative path for urdf files

* changed fileoutput to create directory if necessary

* more math implementation in DefDict and fixed add behavior

File: sim/robots/scalear_leg/urdf_scalar/urdf/scalar.urdf (robot description, URDF)
Before this commit: robot SCALAR, 33 links, 32 joints
Links:
- link A_Link0: geometry collision mesh filename=A_Link0.STL; visual mesh filename=A_Link0.STL
- link A_Link1: geometry collision mesh filename=A_Link1.STL; visual mesh filename=A_Link1.STL
- link A_Link2: geometry collision mesh filename=A_Link2.STL; visual mesh filename=A_Link2.STL
- link A_Link3: geometry collision mesh filename=A_Link3.STL; visual mesh filename=A_Link3.STL
- link B_Link0: geometry collision mesh filename=B_Link0.STL; visual mesh filename=B_Link0.STL
- link B_Link1: geometry collision mesh filename=B_Link1.STL; visual mesh filename=B_Link1.STL
- link B_Link2: geometry collision mesh filename=B_Link2.STL; visual mesh filename=B_Link2.STL
- link B_Link3: geometry collision mesh filename=B_Link3.STL; visual mesh filename=B_Link3.STL
- link E_Link0: geometry collision mesh filename=E_Link0.STL; visual mesh filename=E_Link0.STL
- link E_Link1: geometry collision mesh filename=E_Link1.STL; visual mesh filename=E_Link1.STL
- link E_Link2: geometry collision mesh filename=E_Link2.STL; visual mesh filename=E_Link2.STL
- link E_Link3: geometry collision mesh filename=E_Link3.STL; visual mesh filename=E_Link3.STL
- link F_Link0: geometry collision mesh filename=F_Link0.STL; visual mesh filename=F_Link0.STL
- link F_Link1: geometry collision mesh filename=F_Link1.STL; visual mesh filename=F_Link1.STL
- link F_Link2: geometry collision mesh filename=F_Link2.STL; visual mesh filename=F_Link2.STL
- link F_Link3: geometry collision mesh filename=F_Link3.STL; visual mesh filename=F_Link3.STL
- link Shoulder_Link0: geometry collision mesh filename=Shoulder_Link0.STL; visual mesh filename=Shoulder_Link0.STL
- link Shoulder_Link1: geometry collision mesh filename=Shoulder_Link1.STL; visual mesh filename=Shoulder_Link1.STL
- link Shoulder_Link2: geometry collision mesh filename=Shoulder_Link2.STL; visual mesh filename=Shoulder_Link2.STL
- link Shoulder_Link3: geometry collision mesh filename=Shoulder_Link3.STL; visual mesh filename=Shoulder_Link3.STL
- link body: geometry collision mesh filename=body.STL; visual mesh filename=body.STL

File: sim/robots/scalear_leg/urdf_scalar_6DoF/urdf/SCALAR_6DoF.urdf (robot description, URDF)
Before this commit: robot SCALAR_6DoF, 21 links, 20 joints
Links:
- link A_Link0: geometry collision mesh filename=A_Link0.STL; visual mesh filename=A_Link0.STL
- link A_Link3: geometry collision mesh filename=A_Link3.STL; visual mesh filename=A_Link3.STL
- link B_Link0: geometry collision mesh filename=B_Link0.STL; visual mesh filename=B_Link0.STL
- link B_Link3: geometry collision mesh filename=B_Link3.STL; visual mesh filename=B_Link3.STL
- link E_Link0: geometry collision mesh filename=E_Link0.STL; visual mesh filename=E_Link0.STL
- link E_Link3: geometry collision mesh filename=E_Link3.STL; visual mesh filename=E_Link3.STL
- link F_Link0: geometry collision mesh filename=F_Link0.STL; visual mesh filename=F_Link0.STL
- link F_Link3: geometry collision mesh filename=F_Link3.STL; visual mesh filename=F_Link3.STL
- link Shoulder_Link0: geometry collision mesh filename=Shoulder_Link0.STL; visual mesh filename=Shoulder_Link0.STL
- link Shoulder_Link3: geometry collision mesh filename=Shoulder_Link3.STL; visual mesh filename=Shoulder_Link3.STL
- link body: geometry collision mesh filename=body.STL; visual mesh filename=body.STL
- link wrist1_Link0: geometry collision mesh filename=wrist1_Link0.STL; visual mesh filename=wrist1_Link0.STL
- link wrist1_Link3: geometry collision mesh filename=wrist1_Link3.STL; visual mesh filename=wrist1_Link3.STL
- link wrist2_Link0: geometry collision mesh filename=wrist2_Link0.STL; visual mesh filename=wrist2_Link0.STL
- link wrist2_Link3: geometry collision mesh filename=wrist2_Link3.STL; visual mesh filename=wrist2_Link3.STL
- link wrist3_Link0: geometry collision mesh filename=wrist3_Link0.STL; visual mesh filename=wrist3_Link0.STL
- link wrist3_Link3: geometry collision mesh filename=wrist3_Link3.STL; visual mesh filename=wrist3_Link3.STL
