Commit message: Testing debug, testing immutable, changing process to ray

File: sim/robots/scalear_leg/urdf_scalar_6DoF/urdf/SCALAR_6DoF.urdf (robot description, URDF)
Before this commit: robot SCALAR_6DoF, 21 links, 20 joints
Links:
- link A_Link0: geometry collision mesh filename=/home/yusuke/PycharmProjects/pySiLVIA_lib/AbstractedRobot/s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; visual mesh filename=/home/yusuke/PycharmProjects/pySiLVIA_lib/AbstractedRobot/s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
- link A_Link3: geometry collision mesh filename=/home/yusuke/PycharmProjects/pySiLVIA_lib/AbstractedRobot/s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; visual mesh filename=/home/yusuke/PycharmProjects/pySiLVIA_lib/AbstractedRobot/s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
- link B_Link0: geometry collision mesh filename=/home/yusuke/PycharmProjects/pySiLVIA_lib/AbstractedRobot/s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; visual mesh filename=/home/yusuke/PycharmProjects/pySiLVIA_lib/AbstractedRobot/s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
- link B_Link3: geometry collision mesh filename=/home/yusuke/PycharmProjects/pySiLVIA_lib/AbstractedRobot/s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; visual mesh filename=/home/yusuke/PycharmProjects/pySiLVIA_lib/AbstractedRobot/s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
- link E_Link0: geometry collision mesh filename=/home/yusuke/PycharmProjects/pySiLVIA_lib/AbstractedRobot/s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; visual mesh filename=/home/yusuke/PycharmProjects/pySiLVIA_lib/AbstractedRobot/s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
- link E_Link3: geometry collision mesh filename=/home/yusuke/PycharmProjects/pySiLVIA_lib/AbstractedRobot/s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; visual mesh filename=/home/yusuke/PycharmProjects/pySiLVIA_lib/AbstractedRobot/s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
- link F_Link0: geometry collision mesh filename=/home/yusuke/PycharmProjects/pySiLVIA_lib/AbstractedRobot/s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; visual mesh filename=/home/yusuke/PycharmProjects/pySiLVIA_lib/AbstractedRobot/s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
- link F_Link3: geometry collision mesh filename=/home/yusuke/PycharmProjects/pySiLVIA_lib/AbstractedRobot/s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; visual mesh filename=/home/yusuke/PycharmProjects/pySiLVIA_lib/AbstractedRobot/s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
- link Shoulder_Link0: geometry collision mesh filename=/home/yusuke/PycharmProjects/pySiLVIA_lib/AbstractedRobot/s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; visual mesh filename=/home/yusuke/PycharmProjects/pySiLVIA_lib/AbstractedRobot/s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
- link Shoulder_Link3: geometry collision mesh filename=/home/yusuke/PycharmProjects/pySiLVIA_lib/AbstractedRobot/s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; visual mesh filename=/home/yusuke/PycharmProjects/pySiLVIA_lib/AbstractedRobot/s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
- link body: geometry collision mesh filename=/home/yusuke/PycharmProjects/pySiLVIA_lib/AbstractedRobot/s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; visual mesh filename=/home/yusuke/PycharmProjects/pySiLVIA_lib/AbstractedRobot/s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
- link wrist1_Link0: geometry collision mesh filename=/home/yusuke/PycharmProjects/pySiLVIA_lib/AbstractedRobot/s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; visual mesh filename=/home/yusuke/PycharmProjects/pySiLVIA_lib/AbstractedRobot/s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
- link wrist1_Link3: geometry collision mesh filename=/home/yusuke/PycharmProjects/pySiLVIA_lib/AbstractedRobot/s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; visual mesh filename=/home/yusuke/PycharmProjects/pySiLVIA_lib/AbstractedRobot/s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
- link wrist2_Link0: geometry collision mesh filename=/home/yusuke/PycharmProjects/pySiLVIA_lib/AbstractedRobot/s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; visual mesh filename=/home/yusuke/PycharmProjects/pySiLVIA_lib/AbstractedRobot/s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
- link wrist2_Link3: geometry collision mesh filename=/home/yusuke/PycharmProjects/pySiLVIA_lib/AbstractedRobot/s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; visual mesh filename=/home/yusuke/PycharmProjects/pySiLVIA_lib/AbstractedRobot/s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
- link wrist3_Link0: geometry collision mesh filename=/home/yusuke/PycharmProjects/pySiLVIA_lib/AbstractedRobot/s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; visual mesh filename=/home/yusuke/PycharmProjects/pySiLVIA_lib/AbstractedRobot/s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
- link wrist3_Link3: geometry collision mesh filename=/home/yusuke/PycharmProjects/pySiLVIA_lib/AbstractedRobot/s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; visual mesh filename=/home/yusuke/PycharmProjects/pySiLVIA_lib/AbstractedRobot/s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

Commit message: commit test

File: sim/robots/scalear_leg/urdf_scalar_6DoF/urdf/SCALAR_6DoF.urdf (robot description, URDF)
Before this commit: robot SCALAR_6DoF, 21 links, 20 joints
Links:
- link A_Link0: geometry collision mesh filename=/home/yusuke/PycharmProjects/AbstractedRobot/sim/robots/sca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; visual mesh filename=/home/yusuke/PycharmProjects/AbstractedRobot/sim/robots/sca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
- link A_Link3: geometry collision mesh filename=/home/yusuke/PycharmProjects/AbstractedRobot/sim/robots/sca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; visual mesh filename=/home/yusuke/PycharmProjects/AbstractedRobot/sim/robots/sca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
- link B_Link0: geometry collision mesh filename=/home/yusuke/PycharmProjects/AbstractedRobot/sim/robots/sca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; visual mesh filename=/home/yusuke/PycharmProjects/AbstractedRobot/sim/robots/sca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
- link B_Link3: geometry collision mesh filename=/home/yusuke/PycharmProjects/AbstractedRobot/sim/robots/sca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; visual mesh filename=/home/yusuke/PycharmProjects/AbstractedRobot/sim/robots/sca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
- link E_Link0: geometry collision mesh filename=/home/yusuke/PycharmProjects/AbstractedRobot/sim/robots/sca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; visual mesh filename=/home/yusuke/PycharmProjects/AbstractedRobot/sim/robots/sca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
- link E_Link3: geometry collision mesh filename=/home/yusuke/PycharmProjects/AbstractedRobot/sim/robots/sca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; visual mesh filename=/home/yusuke/PycharmProjects/AbstractedRobot/sim/robots/sca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
- link F_Link0: geometry collision mesh filename=/home/yusuke/PycharmProjects/AbstractedRobot/sim/robots/sca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; visual mesh filename=/home/yusuke/PycharmProjects/AbstractedRobot/sim/robots/sca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
- link F_Link3: geometry collision mesh filename=/home/yusuke/PycharmProjects/AbstractedRobot/sim/robots/sca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; visual mesh filename=/home/yusuke/PycharmProjects/AbstractedRobot/sim/robots/sca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
- link Shoulder_Link0: geometry collision mesh filename=/home/yusuke/PycharmProjects/AbstractedRobot/sim/robots/sca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; visual mesh filename=/home/yusuke/PycharmProjects/AbstractedRobot/sim/robots/sca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
- link Shoulder_Link3: geometry collision mesh filename=/home/yusuke/PycharmProjects/AbstractedRobot/sim/robots/sca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; visual mesh filename=/home/yusuke/PycharmProjects/AbstractedRobot/sim/robots/sca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
- link body: geometry collision mesh filename=/home/yusuke/PycharmProjects/AbstractedRobot/sim/robots/sca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; visual mesh filename=/home/yusuke/PycharmProjects/AbstractedRobot/sim/robots/sca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
- link wrist1_Link0: geometry collision mesh filename=/home/yusuke/PycharmProjects/AbstractedRobot/sim/robots/sca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; visual mesh filename=/home/yusuke/PycharmProjects/AbstractedRobot/sim/robots/sca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
- link wrist1_Link3: geometry collision mesh filename=/home/yusuke/PycharmProjects/AbstractedRobot/sim/robots/sca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; visual mesh filename=/home/yusuke/PycharmProjects/AbstractedRobot/sim/robots/sca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
- link wrist2_Link0: geometry collision mesh filename=/home/yusuke/PycharmProjects/AbstractedRobot/sim/robots/sca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; visual mesh filename=/home/yusuke/PycharmProjects/AbstractedRobot/sim/robots/sca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
- link wrist2_Link3: geometry collision mesh filename=/home/yusuke/PycharmProjects/AbstractedRobot/sim/robots/sca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; visual mesh filename=/home/yusuke/PycharmProjects/AbstractedRobot/sim/robots/sca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
- link wrist3_Link0: geometry collision mesh filename=/home/yusuke/PycharmProjects/AbstractedRobot/sim/robots/sca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; visual mesh filename=/home/yusuke/PycharmProjects/AbstractedRobot/sim/robots/sca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
- link wrist3_Link3: geometry collision mesh filename=/home/yusuke/PycharmProjects/AbstractedRobot/sim/robots/sca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; visual mesh filename=/home/yusuke/PycharmProjects/AbstractedRobot/sim/robots/sca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

Commit message: changed to use relative path for urdf files

File: sim/robots/scalear_leg/urdf_scalar_6DoF/urdf/SCALAR_6DoF.urdf (robot description, URDF)
Before this commit: robot SCALAR_6DoF, 21 links, 20 joints
Links:
- link A_Link0: geometry collision mesh filename=A_Link0.STL; visual mesh filename=A_Link0.STL
- link A_Link3: geometry collision mesh filename=A_Link3.STL; visual mesh filename=A_Link3.STL
- link B_Link0: geometry collision mesh filename=B_Link0.STL; visual mesh filename=B_Link0.STL
- link B_Link3: geometry collision mesh filename=B_Link3.STL; visual mesh filename=B_Link3.STL
- link E_Link0: geometry collision mesh filename=E_Link0.STL; visual mesh filename=E_Link0.STL
- link E_Link3: geometry collision mesh filename=E_Link3.STL; visual mesh filename=E_Link3.STL
- link F_Link0: geometry collision mesh filename=F_Link0.STL; visual mesh filename=F_Link0.STL
- link F_Link3: geometry collision mesh filename=F_Link3.STL; visual mesh filename=F_Link3.STL
- link Shoulder_Link0: geometry collision mesh filename=Shoulder_Link0.STL; visual mesh filename=Shoulder_Link0.STL
- link Shoulder_Link3: geometry collision mesh filename=Shoulder_Link3.STL; visual mesh filename=Shoulder_Link3.STL
- link body: geometry collision mesh filename=body.STL; visual mesh filename=body.STL
- link wrist1_Link0: geometry collision mesh filename=wrist1_Link0.STL; visual mesh filename=wrist1_Link0.STL
- link wrist1_Link3: geometry collision mesh filename=wrist1_Link3.STL; visual mesh filename=wrist1_Link3.STL
- link wrist2_Link0: geometry collision mesh filename=wrist2_Link0.STL; visual mesh filename=wrist2_Link0.STL
- link wrist2_Link3: geometry collision mesh filename=wrist2_Link3.STL; visual mesh filename=wrist2_Link3.STL
- link wrist3_Link0: geometry collision mesh filename=wrist3_Link0.STL; visual mesh filename=wrist3_Link0.STL
- link wrist3_Link3: geometry collision mesh filename=wrist3_Link3.STL; visual mesh filename=wrist3_Link3.STL
