Commit message: SimScaler implementation

File: sim/robots/scaler/pybullet/urdf_scalar/urdf/scalar.urdf (robot description, URDF)
Before this commit: robot SCALAR, 36 links, 35 joints
Links:
- link A_Link0: geometry collision mesh filename=A_Link0.STL; visual mesh filename=A_Link0.STL
- link A_Link1: geometry collision mesh filename=A_Link1.STL; visual mesh filename=A_Link1.STL
- link A_Link2: geometry collision mesh filename=A_Link2.STL; visual mesh filename=A_Link2.STL
- link A_Link3: geometry collision mesh filename=A_Link3.STL; visual mesh filename=A_Link3.STL
- link B_Link0: geometry collision mesh filename=B_Link0.STL; visual mesh filename=B_Link0.STL
- link B_Link1: geometry collision mesh filename=B_Link1.STL; visual mesh filename=B_Link1.STL
- link B_Link2: geometry collision mesh filename=B_Link2.STL; visual mesh filename=B_Link2.STL
- link B_Link3: geometry collision mesh filename=B_Link3.STL; visual mesh filename=B_Link3.STL
- link BodyBot_Link: geometry collision mesh filename=BodyBot_Link.STL; visual mesh filename=BodyBot_Link.STL
- link BodyLeft_Link: geometry collision mesh filename=BodyLeft_Link.STL; visual mesh filename=BodyLeft_Link.STL
- link BodyRight_Link: geometry collision mesh filename=BodyRight_Link.STL; visual mesh filename=BodyRight_Link.STL
- link BodyTopleft_Link: geometry collision mesh filename=BodyTopleft_Link.STL; visual mesh filename=BodyTopleft_Link.STL
- link E_Link0: geometry collision mesh filename=E_Link0.STL; visual mesh filename=E_Link0.STL
- link E_Link1: geometry collision mesh filename=E_Link1.STL; visual mesh filename=E_Link1.STL
- link E_Link2: geometry collision mesh filename=E_Link2.STL; visual mesh filename=E_Link2.STL
- link E_Link3: geometry collision mesh filename=E_Link3.STL; visual mesh filename=E_Link3.STL
- link F_Link0: geometry collision mesh filename=F_Link0.STL; visual mesh filename=F_Link0.STL
- link F_Link1: geometry collision mesh filename=F_Link1.STL; visual mesh filename=F_Link1.STL
- link F_Link2: geometry collision mesh filename=F_Link2.STL; visual mesh filename=F_Link2.STL
- link F_Link3: geometry collision mesh filename=F_Link3.STL; visual mesh filename=F_Link3.STL
- link Shoulder_Link0: geometry collision mesh filename=Shoulder_Link0.STL; visual mesh filename=Shoulder_Link0.STL
- link Shoulder_Link1: geometry collision mesh filename=Shoulder_Link1.STL; visual mesh filename=Shoulder_Link1.STL
- link Shoulder_Link2: geometry collision mesh filename=Shoulder_Link2.STL; visual mesh filename=Shoulder_Link2.STL
- link Shoulder_Link3: geometry collision mesh filename=Shoulder_Link3.STL; visual mesh filename=Shoulder_Link3.STL

File: sim/robots/scaler/pybullet/urdf_scalar_6DoF/urdf/SCALAR_6DoF.urdf (robot description, URDF)
Before this commit: robot SCALAR_6DoF, 44 links, 43 joints
Links:
- link A_Link0: geometry collision mesh filename=A_Link0.STL; visual mesh filename=A_Link0.STL
- link A_Link1: geometry collision mesh filename=A_Link1.STL; visual mesh filename=A_Link1.STL
- link A_Link2: geometry collision mesh filename=A_Link2.STL; visual mesh filename=A_Link2.STL
- link A_Link3: geometry collision mesh filename=A_Link3.STL; visual mesh filename=A_Link3.STL
- link B_Link0: geometry collision mesh filename=B_Link0.STL; visual mesh filename=B_Link0.STL
- link B_Link1: geometry collision mesh filename=B_Link1.STL; visual mesh filename=B_Link1.STL
- link B_Link2: geometry collision mesh filename=B_Link2.STL; visual mesh filename=B_Link2.STL
- link B_Link3: geometry collision mesh filename=B_Link3.STL; visual mesh filename=B_Link3.STL
- link BodyBot_Link: geometry collision mesh filename=BodyBot_Link.STL; visual mesh filename=BodyBot_Link.STL
- link BodyLeft_Link: geometry collision mesh filename=BodyLeft_Link.STL; visual mesh filename=BodyLeft_Link.STL
- link BodyRight_Link: geometry collision mesh filename=BodyRight_Link.STL; visual mesh filename=BodyRight_Link.STL
- link BodyTopleft_Link: geometry collision mesh filename=BodyTopleft_Link.STL; visual mesh filename=BodyTopleft_Link.STL
- link E_Link0: geometry collision mesh filename=E_Link0.STL; visual mesh filename=E_Link0.STL
- link E_Link1: geometry collision mesh filename=E_Link1.STL; visual mesh filename=E_Link1.STL
- link E_Link2: geometry collision mesh filename=E_Link2.STL; visual mesh filename=E_Link2.STL
- link E_Link3: geometry collision mesh filename=E_Link3.STL; visual mesh filename=E_Link3.STL
- link F_Link0: geometry collision mesh filename=F_Link0.STL; visual mesh filename=F_Link0.STL
- link F_Link1: geometry collision mesh filename=F_Link1.STL; visual mesh filename=F_Link1.STL
- link F_Link2: geometry collision mesh filename=F_Link2.STL; visual mesh filename=F_Link2.STL
- link F_Link3: geometry collision mesh filename=F_Link3.STL; visual mesh filename=F_Link3.STL
- link Shoulder_Link0: geometry collision mesh filename=Shoulder_Link0.STL; visual mesh filename=Shoulder_Link0.STL
- link Shoulder_Link1: geometry collision mesh filename=Shoulder_Link1.STL; visual mesh filename=Shoulder_Link1.STL
- link Shoulder_Link2: geometry collision mesh filename=Shoulder_Link2.STL; visual mesh filename=Shoulder_Link2.STL
- link Shoulder_Link3: geometry collision mesh filename=Shoulder_Link3.STL; visual mesh filename=Shoulder_Link3.STL
- link wrist1_Link0: geometry collision mesh filename=wrist1_Link0.STL; visual mesh filename=wrist1_Link0.STL
- link wrist1_Link1: geometry collision mesh filename=wrist1_Link1.STL; visual mesh filename=wrist1_Link1.STL
- link wrist1_Link2: geometry collision mesh filename=wrist1_Link2.STL; visual mesh filename=wrist1_Link2.STL
- link wrist1_Link3: geometry collision mesh filename=wrist1_Link3.STL; visual mesh filename=wrist1_Link3.STL
- link wrist2_Link0: geometry collision mesh filename=wrist2_Link0.STL; visual mesh filename=wrist2_Link0.STL
- link wrist2_Link1: geometry collision mesh filename=wrist2_Link1.STL; visual mesh filename=wrist2_Link1.STL
- link wrist2_Link2: geometry collision mesh filename=wrist2_Link2.STL; visual mesh filename=wrist2_Link2.STL
- link wrist2_Link3: geometry collision mesh filename=wrist2_Link3.STL; visual mesh filename=wrist2_Link3.STL
- link wrist3_Link0: geometry collision mesh filename=wrist3_Link0.STL; visual mesh filename=wrist3_Link0.STL
- link wrist3_Link1: geometry collision mesh filename=wrist3_Link1.STL; visual mesh filename=wrist3_Link1.STL
- link wrist3_Link2: geometry collision mesh filename=wrist3_Link2.STL; visual mesh filename=wrist3_Link2.STL
- link wrist3_Link3: geometry collision mesh filename=wrist3_Link3.STL; visual mesh filename=wrist3_Link3.STL
